File: RF24 Node.brd (EAGLE design)
At the start: 50.2 x 28.6 mm, 27 parts, among them IC1 ATMEGA328P, Q1 16MHz

Commit message: RF24 Node v1.2
Parts:
- removed LM1117: (no value), lm1117:TO220V
- added LM1117T: (no value), lm1117:TO220V
- added REGJMP: (no value), SparkFun-Connectors:1X02
- added U$2: (no value), SparkFun-Aesthetics:OSHW-LOGO-S
- moved A4 3.81 mm to (15.9, 21.6), turned to 180 degrees
- moved D2 0.64 mm to (8.26, 7.62)
- moved D3 0.63 mm to (14.0, 7.62)
- moved PWR 0.63 mm to (2.54, 21.6), turned to 0 degrees
Connections:
- new net N$5: LM1117T.3, REGJMP.2
- net EXTPWR: now also REGJMP.1; no longer LM1117.3
- net GND: now also LM1117T.1; no longer LM1117.1
- net N$1: now also LM1117T.2; no longer LM1117.2
Routing:
- net N$5: track 0.00 -> 11.0 mm
- net RESET: track 52.8 -> 46.9 mm
- net AIN4: track 7.67 -> 3.18 mm
- net +3V3: track 72.4 -> 76.2 mm
- net D13: track 22.7 -> 26.2 mm
- net N$1: track 16.2 -> 19.3 mm
- net D11: track 18.4 -> 19.5 mm
- net D4: track 13.4 -> 14.5 mm
- net GND: track 120.9 -> 121.8 mm
- net D10: track 9.09 -> 9.98 mm
- net D5: track 11.8 -> 12.7 mm
- net EXTPWR: track 28.4 -> 27.7 mm
- net N$2: track 14.0 -> 13.5 mm
- net D7: track 34.3 -> 34.1 mm, vias 2 -> 0
- net N$3: track 13.4 -> 13.2 mm, vias 1 -> 0
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Other:
- board text added: "PWR"
- board text added: "RF24 Node v1.2"
- board text removed: "RF24 Node v1.1"

Commit message: RF24 Node 1.3
Parts:
- added R2: 4K7, resistor:0204V
- added U$1: (no value), SparkFun-Aesthetics:OSHW-LOGO-S
- moved JP1 1.27 mm to (47.0, 25.4)
- moved JP9 0.64 mm to (47.0, 3.17), turned to 90 degrees
- moved JP2 0.64 mm to (3.17, 3.17)
- moved JP8 0.64 mm to (3.17, 25.4)
- moved U$2 0.63 mm to (12.1, 14.6)
Connections:
- net +3V3: now also R2.2
- net D5: now also R2.1
Routing:
- net D6: track 35.6 -> 48.0 mm
- net GND: track 121.8 -> 118.9 mm
- net D12: track 21.5 -> 22.4 mm
Other:
- board text added: "RF24 Node v1.3"
- board text removed: "RF24 Node v1.2"
