File: RF24 Node.sch (EAGLE design)
At the start: 25 parts, among them IC1 ATMEGA328P, Q1 16MHz

Commit message: RF24 Node v1.2
Parts:
- added REGJMP: M02PTH, SparkFun-Connectors:M02PTH
- renumbered LM1117 to LM1117T
Connections:
- new net N$5: LM1117T.IN, REGJMP.2
- net EXTPWR: now also REGJMP.1; no longer LM1117T.IN
Other:
- moved on the sheet: D3
Changed lines of the file:
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@@
 <part name="SUPPLY5" library="supply2" deviceset="GND" device=""/>
 <part name="DS18B20" library="Ava" deviceset="DS1820" device="TO92" value=""/>
-<part name="LM1117" library="lm1117" deviceset="LM1117T-*" device="-V" technology="3.3" value=""/>
+<part name="LM1117T" library="lm1117" deviceset="LM1117T-*" device="-V" technology="3.3" value=""/>
+<part name="REGJMP" library="SparkFun-Connectors" deviceset="M02" device="PTH" value=""/>
 <part name="D3" library="SparkFun-Connectors" deviceset="M02" device="PTH" value=""/>
 <part name="SUPPLY6" library="supply2" deviceset="GND" device=""/>
@@
 <instance part="SUPPLY5" gate="GND" x="60.96" y="119.38" rot="R90"/>
 <instance part="DS18B20" gate="G$1" x="53.34" y="76.2" rot="MR90"/>
-<instance part="LM1117" gate="G$1" x="93.98" y="127"/>
-<instance part="D3" gate="G$1" x="50.8" y="88.9"/>
-<instance part="SUPPLY6" gate="GND" x="60.96" y="88.9" rot="R90"/>
+<instance part="LM1117T" gate="G$1" x="93.98" y="127"/>
+<instance part="REGJMP" gate="G$1" x="76.2" y="111.76"/>
+<instance part="D3" gate="G$1" x="50.8" y="91.44"/>
+<instance part="SUPPLY6" gate="GND" x="60.96" y="91.44" rot="R90"/>
 </instances>
 <busses>
@@
 </segment>
 <segment>
-<pinref part="LM1117" gate="G$1" pin="GND"/>
+<pinref part="LM1117T" gate="G$1" pin="GND"/>
 <pinref part="SUPPLY10" gate="GND" pin="GND"/>
 </segment>
@@
 <pinref part="SW_PWR" gate="BEF1" pin="O"/>
 <wire x1="101.6" y1="104.14" x2="101.6" y2="111.76" width="0.1524" layer="91"/>
+<junction x="101.6" y="104.14"/>
+<pinref part="REGJMP" gate="G$1" pin="1"/>
 <wire x1="101.6" y1="111.76" x2="83.82" y2="111.76" width="0.1524" layer="91"/>
-<wire x1="83.82" y1="111.76" x2="83.82" y2="127" width="0.1524" layer="91"/>
-<pinref part="LM1117" gate="G$1" pin="IN"/>
-<wire x1="83.82" y1="127" x2="86.36" y2="127" width="0.1524" layer="91"/>
-<junction x="101.6" y="104.14"/>
 </segment>
 </net>
@@
 </segment>
 </net>
-<net name="D3" class="0">
-<segment>
-<pinref part="IC1" gate="1" pin="PD3(INT1/OC2B/PCINT19)"/>
-<wire x1="-30.48" y1="43.18" x2="-17.78" y2="43.18" width="0.1524" layer="91"/>
-<label x="-27.94" y="43.18" size="1.778" layer="95"/>
-</segment>
-<segment>
-<pinref part="D3" gate="G$1" pin="2"/>
-<wire x1="58.42" y1="91.44" x2="60.96" y2="91.44" width="0.1524" layer="91"/>
-<label x="60.96" y="91.44" size="1.778" layer="95"/>
-</segment>
-</net>
 <net name="D6" class="0">
 <segment>
@@
 <net name="N$1" class="0">
 <segment>
-<pinref part="LM1117" gate="G$1" pin="OUT"/>
+<pinref part="LM1117T" gate="G$1" pin="OUT"/>
 <wire x1="101.6" y1="127" x2="109.22" y2="127" width="0.1524" layer="91"/>
 <wire x1="109.22" y1="127" x2="109.22" y2="124.46" width="0.1524" layer="91"/>
@@
 </segment>
 </net>
+<net name="N$5" class="0">
+<segment>
+<pinref part="REGJMP" gate="G$1" pin="2"/>
+<wire x1="83.82" y1="114.3" x2="83.82" y2="127" width="0.1524" layer="91"/>
+<pinref part="LM1117T" gate="G$1" pin="IN"/>
+<wire x1="83.82" y1="127" x2="86.36" y2="127" width="0.1524" layer="91"/>
+</segment>
+</net>
+<net name="D3" class="0">
+<segment>
+<pinref part="IC1" gate="1" pin="PD3(INT1/OC2B/PCINT19)"/>
+<wire x1="-30.48" y1="43.18" x2="-17.78" y2="43.18" width="0.1524" layer="91"/>
+<label x="-27.94" y="43.18" size="1.778" layer="95"/>
+</segment>
+<segment>
+<pinref part="D3" gate="G$1" pin="2"/>
+<wire x1="58.42" y1="93.98" x2="60.96" y2="93.98" width="0.1524" layer="91"/>
+<label x="58.42" y="93.98" size="1.778" layer="95"/>
+</segment>
+</net>

Commit message: RF24 Node 1.3
Parts:
- added R2: 4K7, resistor:R-US_0204/2V
Connections:
- net +3V3: now also R2.2
- net D5: now also R2.1
Changed lines of the file:
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@@
 <part name="D3" library="SparkFun-Connectors" deviceset="M02" device="PTH" value=""/>
 <part name="SUPPLY6" library="supply2" deviceset="GND" device=""/>
+<part name="R2" library="resistor" deviceset="R-US_" device="0204/2V" value="4K7"/>
 </parts>
 <sheets>
@@
 <instance part="D3" gate="G$1" x="50.8" y="91.44"/>
 <instance part="SUPPLY6" gate="GND" x="60.96" y="91.44" rot="R90"/>
+<instance part="R2" gate="G$1" x="17.78" y="78.74" rot="R90"/>
 </instances>
 <busses>
@@
 <pinref part="DS18B20" gate="G$1" pin="VCC"/>
 <wire x1="27.94" y1="78.74" x2="48.26" y2="78.74" width="0.1524" layer="91"/>
+<pinref part="R2" gate="G$1" pin="2"/>
+<wire x1="27.94" y1="78.74" x2="30.48" y2="78.74" width="0.1524" layer="91"/>
+<wire x1="30.48" y1="78.74" x2="17.78" y2="83.82" width="0.1524" layer="91"/>
 </segment>
 <segment>
@@
 <wire x1="48.26" y1="76.2" x2="38.1" y2="76.2" width="0.1524" layer="91"/>
 <label x="38.1" y="76.2" size="1.778" layer="95"/>
-</segment>
-</net>
+<pinref part="R2" gate="G$1" pin="1"/>
+<wire x1="38.1" y1="76.2" x2="30.48" y2="76.2" width="0.1524" layer="91"/>
+<wire x1="30.48" y1="76.2" x2="17.78" y2="73.66" width="0.1524" layer="91"/>
+<junction x="38.1" y="76.2"/>
+</segment>
+</net>
